File: hardware/Kicad/Servo Tester/Servo Tester.kicad_sch (KiCad schematic)
At the start: 0 parts

Commit message: Update sweep settings and ignore KiCad lock/cache artifacts
Parts:
- added A1: Clone_Pro_Mini_Socket, PCM_arduino-library:Clone_Pro_Mini_Socket, symbol PCM_arduino-library:Clone_Pro_Mini_Socket
- added BT1: BK-18650-PC4, CodeWorks-Essentials:BAT_BK-18650-PC4, symbol CodeWorks Essentials:BK-18650-PC4
- added C1, C3, C4: 0.1uF, Capacitor_SMD:C_0603_1608Metric, symbol Device:C
- added C2: 0.1uf, Capacitor_SMD:C_0603_1608Metric, symbol Device:C
- added C5: 10uF, Capacitor_SMD:C_0603_1608Metric, symbol Device:C
- added C6: 100nF, Capacitor_SMD:C_0603_1608Metric, symbol Device:C
- added D1: LED, LED_THT:LED_D3.0mm, symbol Device:LED
- added F1: Polyfuse, Fuse:Fuse_Bourns_MF-RG300, symbol Device:Polyfuse
- added J1: Servo 2, Connector_PinHeader_2.54mm:PinHeader_1x03_P2.54mm_Vertical, symbol Connector:Conn_01x03_Pin
- added J2: Servo 3, Connector_PinHeader_2.54mm:PinHeader_1x03_P2.54mm_Vertical, symbol Connector:Conn_01x03_Pin
- added J3: Servo 1, Connector_PinHeader_2.54mm:PinHeader_1x03_P2.54mm_Vertical, symbol Connector:Conn_01x03_Pin
- added OLED1: ~, CodeWorks-Essentials:OLED_0.96_SPI_Module_1x07_P2.54mm, symbol CodeWorks Essentials:OLED_096_SPI
- added R1, R2, R4, R5, R7, R8: 10R, Resistor_SMD:R_0603_1608Metric, symbol Device:R
- added R10, R11: 4.7K, Resistor_SMD:R_0603_1608Metric, symbol Device:R
- added R12: 330R, Resistor_SMD:R_0603_1608Metric, symbol Device:R
- added R13: 47K, Resistor_SMD:R_0603_1608Metric, symbol Device:R
- added R14: 27K, Resistor_SMD:R_0603_1608Metric, symbol Device:R
- added R15: 470R, Resistor_SMD:R_0603_1608Metric, symbol Device:R
- added R3, R6, R9: 0.1R, Resistor_SMD:R_1210_3225Metric, symbol Device:R
- added RV2: 10K, Potentiometer_THT:Potentiometer_Bourns_PTV09A-1_Single_Vertical, symbol Device:R_Potentiometer
- added SW1: SW_Push - Select, Button_Switch_THT:SW_PUSH_6mm, symbol Switch:SW_Push
- added SW2: SW_Push - Down, Button_Switch_THT:SW_PUSH_6mm, symbol Switch:SW_Push
- added SW3: SW_Push - Up, Button_Switch_THT:SW_PUSH_6mm, symbol Switch:SW_Push
- added SW4: HV (8,4V) / STD (5V), Button_Switch_THT:SW_XKB_DM1-16UD-1, symbol Switch:SW_SPDT_321
- added SW5: ON/OFF, symbol Switch:SW_SPST
- added U1: INA3221, Package_DFN_QFN:Texas_RGV0016A_VQFN-16-1EP_4x4mm_P0.65mm_EP2.1x2.1mm, symbol Power_Management:INA3221
- added U2: Mini360, CodeWorks-Essentials:Ultra Mini-360, symbol CodeWorks Essentials:Mini360
Connections:
- new net: C2.1, R4.1, U1.15 (IN+2)
- new net: D1.2 (A), R15.1
- new net: C2.2, R5.1, U1.14 (IN-2)
- new net: C3.2, R8.1, U1.1 (IN-3)
- new net: C3.1, R7.1, U1.2 (IN+3)
- new net: C1.1, R2.1, U1.12 (IN+1)
- new net: C1.2, R1.1, U1.11 (IN-1)
- new net: SW4.3 (A), SW5.2 (B), U2.2 (IN+)
- new net: BT1.1+, F1.1
- new net: F1.2, SW5.1 (A)
- new net: BT1.1-, BT1.2+
- new net +5V: A1.Vcc1 (Vcc), C4.1, C5.1, C6.1, OLED1.2 (VCC), R10.2, R11.2, RV2.1, SW4.1 (C), U1.16 (VPU), U2.4 (OUT+)
- new net +BATT: J1.2 (Pin_2), J2.2 (Pin_2), J3.2 (Pin_2), R13.2, SW4.2 (B)
- new net ALERT LED: A1.D4, R15.2
- new net BTN - DOWN: A1.D3 (D3_INT1), SW2.2
- new net BTN - SELECT: A1.D5, SW1.2
- new net BTN - UP: A1.D2 (D2_INT0), SW3.2
- new net GND: A1.GND1 (GND), A1.GND2 (GND), A1.GND3 (GND), BT1.2-, C4.2, C5.2, C6.2, D1.1 (K), J1.3 (Pin_3), J2.3 (Pin_3), J3.3 (Pin_3), OLED1.1 (GND), R1.2, R14.1, R2.2, R3.1, R3.2, R4.2, R5.2, R6.1, R6.2, R7.2, R8.2, R9.1, R9.2, RV2.3, SW1.1, SW2.1, SW3.1, U1.3 (GND), U2.1 (IN-), U2.3 (OUT-)
- new net OLED CLK: A1.D10 (D10_CS), OLED1.3 (SCK)
- new net OLED CS: A1.D12 (D12_MISO), OLED1.7 (CS)
- new net OLED DC: A1.D11 (D11_MOSI), OLED1.6 (DC)
- new net OLED MOSI: A1.D9, OLED1.4 (MOSI)
- new net OLED RST: A1.D13 (D13_SCK), OLED1.5 (RES)
- new net POT: A1.A0, RV2.2
- new net RAIL V: A1.A1, R13.1, R14.2
- new net SCL: A1.A5 (A5/SCL), R11.1, U1.6 (SCL)
- new net SDA: A1.A4 (A4/SDA), R10.1, U1.7 (SDA)
- new net SERVO-SIG: A1.D6, J1.1 (Pin_1), J2.1 (Pin_1), J3.1 (Pin_1), R12.1, R12.2
Other:
- note added: "Arduino PRO MINI"
- note added: "CURRENT MEASUREMENT"
- note added: "Controls"
- note added: "LCD"
- note added: "POWER"
- company: (none) -> CodeWorks  - Michal Pavlik
- title: (none) -> Servo Tester
