File: hardware/Kicad/Servo Tester/Servo Tester.kicad_sch (KiCad schematic)
At the start: 58 parts, among them J1 Servo 1, J2 Servo 2, J3 Servo 3, J4 XT60PW-M, SW1 SS-12D11, SW2 STD / HV, SW3 SW_Push - Up, SW4 SW_Push - Select, SW5 SW_Push - Down, U1 Mini360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

Commit message: Add designators, netlist, positions, and symbol library for Servo Tester project
- Created designators.csv to define component designators for the Servo Tester.
- Added netlist.ipc to specify the electrical connections and layout of the circuit.
- Introduced positions.csv to provide the coordinates and rotation for each component on the PCB.
- Established sym-lib-table to include the Servo Tester symbol library in KiCad.
Parts:
- removed J4: XT60PW-M, Connector_AMASS:AMASS_XT60IPW-M_1x03_P7.20mm_Horizontal, symbol CodeWorks-Connectors:XT60PW-M
- removed SW1: SS-12D11, CodeWorks-Essentials:SS-12D11, symbol CodeWorks Essentials:SS-12D11
- removed SW2: STD / HV, CodeWorks-Essentials:SS-12D10, symbol CodeWorks Essentials:SS-12D11
- added J4: XT60PW-M, CodeWorks-Connectors:AMASS_XT60PW-M_1x02_P7.20mm_Horizontal, symbol Servo Tester:XT60PW-M
- added MH6: (no value), MountingHole:MountingHole_3.2mm_M3_Pad_Via, symbol Servo Tester:MountingHole_Pad
- added SW1: SS-12DXX, CodeWorks-Slide_Switches:SS12D11, symbol Servo Tester:SS-12DXX
- added SW2: SS-12DXX, CodeWorks-Slide_Switches:SS12D10, symbol Servo Tester:SS-12DXX
- A1: symbol PCM_arduino-library:Clone_Pro_Mini_Socket -> Servo Tester:Clone_Pro_Mini_Socket
- BATT1: value BATT -> TestPoint; symbol Connector:TestPoint -> Servo Tester:TestPoint
- BT1: symbol CodeWorks Essentials:BK-18650-PC4 -> Servo Tester:BK-18650-PC4
- C1, C2, C5: value 100nF -> C; symbol Device:C -> Servo Tester:C
- C3, C6, C8: value 0.1uF -> C; symbol Device:C -> Servo Tester:C
- C4: value 10uF -> C; symbol Device:C -> Servo Tester:C
- C7: value 0.1uf -> C; symbol Device:C -> Servo Tester:C
- D1: value STD -> LED; symbol Device:LED -> Servo Tester:LED
- D2: value HV -> LED; symbol Device:LED -> Servo Tester:LED
- D3: value ALERT -> LED; symbol Device:LED -> Servo Tester:LED
- F1: value Polyfuse - 3A -> Polyfuse 3A; footprint Fuse:Fuse_Bourns_MF-RG300 -> CodeWorks-Essentials:Fuse_LittleFuseRUEF300; symbol Device:Polyfuse -> Servo Tester:Polyfuse
- GND1: value GND -> TestPoint; symbol Connector:TestPoint -> Servo Tester:TestPoint
- J1: value Servo 1 -> Conn_01x03_Pin; symbol Connector:Conn_01x03_Pin -> Servo Tester:Conn_01x03_Pin
- J2: value Servo 2 -> Conn_01x03_Pin; symbol Connector:Conn_01x03_Pin -> Servo Tester:Conn_01x03_Pin
- J3: value Servo 3 -> Conn_01x03_Pin; symbol Connector:Conn_01x03_Pin -> Servo Tester:Conn_01x03_Pin
- JP2: value 5V -> SolderJumper_2_Open; symbol Jumper:SolderJumper_2_Open -> Servo Tester:SolderJumper_2_Open
- MH1, MH2, MH3, MH4, MH5: value M3 -> (none); symbol Mechanical:MountingHole_Pad -> Servo Tester:MountingHole_Pad
- OLED1: value ~ -> (none); symbol CodeWorks Essentials:OLED_096_SPI -> Servo Tester:OLED_096_SPI
- R1: value 47K -> R; symbol Device:R -> Servo Tester:R
- R10, R11, R12, R13, R14, R15: value 10R -> R; symbol Device:R -> Servo Tester:R
- R16, R17, R18: value 0.1R -> R; symbol Device:R -> Servo Tester:R
- R2: value 27K -> R; symbol Device:R -> Servo Tester:R
- R3: value 0R -> R; symbol Device:R -> Servo Tester:R
- R4, R5: value 1K -> R; symbol Device:R -> Servo Tester:R
- R6: value 470R -> R; symbol Device:R -> Servo Tester:R
- R7, R8: value 4.7K -> R; symbol Device:R -> Servo Tester:R
- R9: value 330R -> R; symbol Device:R -> Servo Tester:R
- RAIL-V1: value ~ -> TestPoint; symbol Connector:TestPoint -> Servo Tester:TestPoint
- RV1: footprint Potentiometer_THT:Potentiometer_Bourns_PTV09A-1_Single_Vertical -> CodeWorks-Potentiometers:Potentiometer_Bourns_PTV09A-1_Single_Vertical; symbol Device:R_Potentiometer -> Servo Tester:R_Potentiometer
- SCL1: value SCL -> TestPoint; symbol Connector:TestPoint -> Servo Tester:TestPoint
- SDA1: value SDA -> TestPoint; symbol Connector:TestPoint -> Servo Tester:TestPoint
- SERVO-SIG1: value SERVO-SIG -> TestPoint; symbol Connector:TestPoint -> Servo Tester:TestPoint
- SW3: value SW_Push - Up -> SW_Push - Down; footprint Button_Switch_THT:SW_PUSH_6mm_H8.5mm -> CodeWorks-Tactile_Switches:SW_PUSH_6mm_H8.5mm; symbol Switch:SW_Push -> Servo Tester:SW_Push
- SW4: value SW_Push - Select -> SW_Push - Down; footprint Button_Switch_THT:SW_PUSH_6mm_H8.5mm -> CodeWorks-Tactile_Switches:SW_PUSH_6mm_H8.5mm; symbol Switch:SW_Push -> Servo Tester:SW_Push
- SW5: footprint Button_Switch_THT:SW_PUSH_6mm_H8.5mm -> CodeWorks-Tactile_Switches:SW_PUSH_6mm_H8.5mm; symbol Switch:SW_Push -> Servo Tester:SW_Push
- U1: symbol CodeWorks Essentials:Mini360 -> Servo Tester:Mini360
- U2: footprint Package_DFN_QFN:Texas_RGV0016A_VQFN-16-1EP_4x4mm_P0.65mm_EP2.1x2.1mm -> CodeWorks-ICs:INA3221_VQFN-16_4x4mm_P0.65mm_EP2.6x2.6mm; symbol Power_Management:INA3221 -> Servo Tester:INA3221
- VPU1: value VPU -> SolderJumper_2_Open; symbol Jumper:SolderJumper_2_Open -> Servo Tester:SolderJumper_2_Open
Connections:
- net +BATT: now also SW2.2
- net GND: now also J4.1 (P), J4.SH1 (SHIELD), J4.SH2 (SHIELD__1), MH6.1
- net at U1.2 (IN+): now also SW1.3, SW2.3
- net at JP2.2 (B), U1.4 (OUT+): now also SW2.1
- net at F1.2: now also SW1.2
- net BATT+: now reaches BT1.1+, F1.1
- net BATT+: now also J4.2 (N)
- net BATT: now reaches BT1.1-, BT1.2+
Other:
- moved on the sheet: JP2, VPU1

Commit message: feat: Add language selection and improve UI for servo tester
- Introduced compile-time language selection for English and Czech.
- Updated UI strings to use language-specific definitions.
- Added support for optional power mode indicator LEDs.
- Implemented burn cycles feature to limit servo sweep cycles.
- Enhanced settings storage and validation for new burn cycles parameter.
- Improved serial debug output for INA3221 communication checks.
- Updated display functions to reflect new settings and language changes.
- Adjusted pin configuration in documentation to match new features.
Parts:
- C1, C2, C5: value C -> 100nF
- C3, C7, C8: value C -> 0.1uF
- C4: value C -> 10uF
- C6: value C -> 0.1nF
- D1: value LED -> STD
- D2: value LED -> HV
- D3: value LED -> ALERT
- J1: value Conn_01x03_Pin -> Servo 1
- J2: value Conn_01x03_Pin -> Servo 2
- J3: value Conn_01x03_Pin -> Servo 3
- R1: value R -> 47K
- R10, R11, R12, R13, R14, R15: value R -> 10R
- R16, R17, R18: value R -> 0.1R
- R2: value R -> 27K
- R3: value R -> 0R
- R4, R5: value R -> 1K
- R6: value R -> 470R
- R7, R8: value R -> 4K7
- R9: value R -> 330R
- SW3: value SW_Push - Down -> SW_Push - Up
- SW4: value SW_Push - Down -> SW_Push - Select
Other:
- moved on the sheet: C6, C7, C8
