File: hardware/kicad/servo_tester/servo_tester.kicad_sch (KiCad schematic)
At the start: 37 parts, among them J1 Servo 2, J2 Servo 3, J3 Servo 1, SW1 SW_Push - Select, SW2 SW_Push - Down, SW3 SW_Push - Up, SW4 HV (8,4V) / STD (5V), SW5 ON/OFF, U1 INA3221, U2 Mini360

Commit message: Update OLED pin mapping and sync hardware files
Parts:
- removed SW4: HV (8,4V) / STD (5V), Button_Switch_THT:SW_XKB_DM1-16UD-1, symbol Switch:SW_SPDT_321
- removed SW5: ON/OFF, symbol Switch:SW_SPST
- added BATT1: BATT, TestPoint:TestPoint_Pad_D2.0mm, symbol Connector:TestPoint
- added C1, C2: 100nF, Capacitor_SMD:C_0805_2012Metric, symbol Device:C
- added D1: STD, LED_THT:LED_D3.0mm, symbol Device:LED
- added D2: HV, LED_THT:LED_D3.0mm, symbol Device:LED
- added GND1: GND, TestPoint:TestPoint_Pad_D2.0mm, symbol Connector:TestPoint
- added J4: XT60PW-M, Connector_AMASS:AMASS_XT60IPW-M_1x03_P7.20mm_Horizontal, symbol CodeWorks-Connectors:XT60PW-M
- added JP2: 5V, Jumper:SolderJumper-2_P1.3mm_Open_RoundedPad1.0x1.5mm, symbol Jumper:SolderJumper_2_Open
- added MH1, MH2, MH3, MH4, MH5: M3, MountingHole:MountingHole_3.2mm_M3_Pad_Via, symbol Mechanical:MountingHole_Pad
- added R3: 0R, Resistor_SMD:R_0805_2012Metric, symbol Device:R
- added R4, R5: 1K, Resistor_SMD:R_0805_2012Metric, symbol Device:R
- added RAIL-V1: ~, TestPoint:TestPoint_Pad_D2.0mm, symbol Connector:TestPoint
- added SCL1: SCL, TestPoint:TestPoint_Pad_D2.0mm, symbol Connector:TestPoint
- added SDA1: SDA, TestPoint:TestPoint_Pad_D2.0mm, symbol Connector:TestPoint
- added SERVO-SIG1: SERVO-SIG, TestPoint:TestPoint_Pad_D2.0mm, symbol Connector:TestPoint
- added SW1: SS-12D11, CodeWorks-Essentials:SS-12D11, symbol CodeWorks Essentials:SS-12D11
- added SW2: STD / HV, CodeWorks-Essentials:SS-12D10, symbol CodeWorks Essentials:SS-12D11
- added VPU1: VPU, Jumper:SolderJumper-2_P1.3mm_Open_RoundedPad1.0x1.5mm, symbol Jumper:SolderJumper_2_Open
- A1: footprint PCM_arduino-library:Clone_Pro_Mini_Socket -> CodeWorks-Essentials:Clone_Pro_Mini_Socket_No_PROG
- C3: renamed from C4; footprint Capacitor_SMD:C_0603_1608Metric -> Capacitor_SMD:C_0805_2012Metric
- C4: renamed from C5; footprint Capacitor_SMD:C_0603_1608Metric -> Capacitor_SMD:C_0805_2012Metric
- C5: renamed from C6; footprint Capacitor_SMD:C_0603_1608Metric -> Capacitor_SMD:C_0805_2012Metric
- C6: renamed from C1; footprint Capacitor_SMD:C_0603_1608Metric -> Capacitor_SMD:C_0805_2012Metric
- C7: renamed from C2; footprint Capacitor_SMD:C_0603_1608Metric -> Capacitor_SMD:C_0805_2012Metric
- C8: renamed from C3; footprint Capacitor_SMD:C_0603_1608Metric -> Capacitor_SMD:C_0805_2012Metric
- D3: renamed from D1; value LED -> ALERT
- F1: value Polyfuse -> Polyfuse - 3A
- J1: renamed from J3; footprint Connector_PinHeader_2.54mm:PinHeader_1x03_P2.54mm_Vertical -> Connector_PinHeader_2.54mm:PinHeader_1x03_P2.54mm_Horizontal
- J2: renamed from J1; footprint Connector_PinHeader_2.54mm:PinHeader_1x03_P2.54mm_Vertical -> Connector_PinHeader_2.54mm:PinHeader_1x03_P2.54mm_Horizontal
- J3: renamed from J2; footprint Connector_PinHeader_2.54mm:PinHeader_1x03_P2.54mm_Vertical -> Connector_PinHeader_2.54mm:PinHeader_1x03_P2.54mm_Horizontal
- R1: renamed from R13; footprint Resistor_SMD:R_0603_1608Metric -> Resistor_SMD:R_0805_2012Metric
- R10: renamed from R2; footprint Resistor_SMD:R_0603_1608Metric -> Resistor_SMD:R_0805_2012Metric
- R11: renamed from R1; footprint Resistor_SMD:R_0603_1608Metric -> Resistor_SMD:R_0805_2012Metric
- R12: renamed from R4; footprint Resistor_SMD:R_0603_1608Metric -> Resistor_SMD:R_0805_2012Metric
- R13: renamed from R5; footprint Resistor_SMD:R_0603_1608Metric -> Resistor_SMD:R_0805_2012Metric
- R14: renamed from R7; footprint Resistor_SMD:R_0603_1608Metric -> Resistor_SMD:R_0805_2012Metric
- R15: renamed from R8; footprint Resistor_SMD:R_0603_1608Metric -> Resistor_SMD:R_0805_2012Metric
- R2: renamed from R14; footprint Resistor_SMD:R_0603_1608Metric -> Resistor_SMD:R_0805_2012Metric
- R6: renamed from R15; footprint Resistor_SMD:R_0603_1608Metric -> Resistor_SMD:R_0805_2012Metric
- R7: renamed from R10; footprint Resistor_SMD:R_0603_1608Metric -> Resistor_SMD:R_0805_2012Metric
- R8: renamed from R11; footprint Resistor_SMD:R_0603_1608Metric -> Resistor_SMD:R_0805_2012Metric
- R9: renamed from R12; footprint Resistor_SMD:R_0603_1608Metric -> Resistor_SMD:R_0805_2012Metric
- SW3: footprint Button_Switch_THT:SW_PUSH_6mm -> Button_Switch_THT:SW_PUSH_6mm_H8.5mm
- SW4: renamed from SW1; footprint Button_Switch_THT:SW_PUSH_6mm -> Button_Switch_THT:SW_PUSH_6mm_H8.5mm
- SW5: renamed from SW2; footprint Button_Switch_THT:SW_PUSH_6mm -> Button_Switch_THT:SW_PUSH_6mm_H8.5mm
- renumbered R3 to R16, R6 to R17, R9 to R18, RV2 to RV1, U2 to U1, U1 to U2
Connections:
- net +5V: now also U2.4 (VS), C1.1, C2.1, JP2.1 (A), VPU1.2 (B); no longer U1.4 (OUT+), U2.16 (VPU)
- net +BATT: now also BATT1.1, SW2.1
- net GND: now also C1.2, C2.2, D1.1 (K), D2.1 (K), GND1.1, J4.1 (P), J4.SH1 (SHIELD), J4.SH2 (SHIELD__1), MH1.1, MH2.1, MH3.1, MH4.1, MH5.1; no longer J1.3 (Pin_3), J2.3 (Pin_3), J3.3 (Pin_3), R10.2, R12.2, R14.2, R16.2, R17.2, R18.2
- net RAIL V: now also R3.1; no longer R1.1, R2.2
- net SCL: now also SCL1.1
- net SDA: now also SDA1.1
- net SERVO-SIG: no longer A1.D6, R9.2
- net IN+2: now reaches C7.1, R12.1, U2.15 (IN+2)
- net STD: now reaches A1.D7
- net STD: now also R4.2
- net HV: now reaches A1.D8
- net HV: now also R5.2
- net IN-2: now reaches C7.2, R13.1, U2.14 (IN-2)
- net IN-3: now reaches C8.2, R15.1, U2.1 (IN-3)
- net IN+3: now reaches C8.1, R14.1, U2.2 (IN+3)
- net IN+1: now reaches C6.1, R10.1, U2.12 (IN+1)
- net IN-1: now reaches C6.2, R11.1, U2.11 (IN-1)
- net at U1.2 (IN+): now also SW1.2, SW2.2
- net at BT1.1+, F1.1: now also J4.2 (N)
- net at F1.2: now also SW1.1
- net ALERT LED renamed ALERT-LED
- net BTN - DOWN renamed BTN-DOWN
- net BTN - SELECT renamed BTN-SELECT
- net BTN - UP renamed BTN-UP
- net OLED CLK renamed OLED-MOSI
- net OLED-MOSI: now also OLED1.4 (MOSI); no longer OLED1.3 (SCK)
- net OLED CS renamed OLED-CS
- net OLED-CS: now also A1.D13 (D13_SCK); no longer A1.D12 (D12_MISO)
- net OLED DC renamed OLED-DC
- net OLED-DC: now also A1.D12 (D12_MISO); no longer A1.D11 (D11_MOSI)
- net OLED MOSI renamed OLED-SCK
- net OLED-SCK: now also OLED1.3 (SCK); no longer OLED1.4 (MOSI)
- net OLED RST renamed OLED-RES
- net OLED-RES: now also A1.D11 (D11_MOSI); no longer A1.D13 (D13_SCK)
- new net: J2.3 (Pin_3), R12.2, R17.2
- new net: R1.1, R2.2, R3.2, RAIL-V1.1
- new net: J3.3 (Pin_3), R14.2, R18.2
- new net: D1.2 (A), R4.1
- new net: J1.3 (Pin_3), R10.2, R16.2
- new net: JP2.2 (B), SW2.3, U1.4 (OUT+)
- new net: D2.2 (A), R5.1
- new net: U2.16 (VPU), VPU1.1 (A)
- new net SERVO: A1.D6, R9.2, SERVO-SIG1.1
- no-connect marks 0 -> 22
Other:
- note added: "MOUNTING HOLES"
- note added: "OLED"
- note added: "OLED 0.96S SPI - 7PIN 1 GND 2 VCC 3 D0 (SPI Clock, SCK) 4 D1 (SPI Data, MOSI) 5 RES 6 DC 7 SC"
- note added: "SERVOS"
- note removed: "LCD"
- moved on the sheet: BT1, D3, F1, R1, R2, R6, RV1, SW3, SW4, SW5
